File: ESP32/Smart Home Energy Management System/Smart Home Energy Management System.kicad_sch (KiCad schematic)
At the start: 0 parts

Commit message: Update from work
Parts:
- added C1, C4: 4.7uF/16V, Capacitor_THT:CP_Radial_D5.0mm_P2.00mm, symbol PCM_SL_Capacitors:4.7uF_16V
- added C10, C11, C12: 0.1uF/25V, Capacitor_SMD:C_0805_2012Metric, symbol SparkFun-Capacitor:0.1uF_0603_25V_20%
- added C2: 10uF_16V, Capacitor_THT:CP_Radial_D5.0mm_P2.00mm, symbol PCM_SL_Capacitors:10uF_16V
- added C3, C5: 100nF, symbol Device:C_Small
- added C6: 470nF, Capacitor_THT:C_Disc_D5.0mm_W2.5mm_P2.50mm, symbol PCM_SL_Capacitors:104_Ceramic
- added C7: 100nF, Capacitor_THT:C_Disc_D5.0mm_W2.5mm_P2.50mm, symbol PCM_SL_Capacitors:104_Ceramic
- added C8, C9: 22pF, symbol Device:C_Small
- added D1, D5: 1N5819, Diode_THT:D_DO-41_SOD81_P10.16mm_Horizontal, symbol Diode:1N5819
- added D10, D11, D12, D13, D14, D15, D16, D17, D18, D6, D7, D8, D9: SM4001, Diode_SMD:D_MELF, symbol Diode:SM4001
- added D2, D4: Red, SparkFun-LED:LED_0603_1608Metric_Red, symbol SparkFun-LED:LED_Red_0603
- added D3: Green, SparkFun-LED:LED_0603_1608Metric_Red, symbol SparkFun-LED:LED_Red_0603
- added J1: USB_C Conn, symbol Connector:Screw_Terminal_01x04
- added J2, J3, J4, J5, J6, J7: LOAD, TerminalBlock_Phoenix:TerminalBlock_Phoenix_PT-1,5-2-5.0-H_1x02_P5.00mm_Horizontal, symbol PCM_SL_Screw_Terminal:Screw_Terminal_2_P5.00mm
- added JP1: ~, SparkFun-Jumper:Jumper_2_NO, symbol SparkFun-Jumper:SolderJumper_2_Open
- added K1, K10, K11, K12, K2, K3, K4, K5, K6, K7, K8, K9: RAYEX-L90, Relay_THT:Relay_SPDT_RAYEX-L90, symbol Relay:RAYEX-L90
- added Q1, Q2: ULN2803ADWR, digikey-footprints:DIP-18_W7.62mm, symbol dk_Transistors-Bipolar-BJT-Arrays:ULN2803ADWR
- added Q3: UMH3N, Package_TO_SOT_SMD:SOT-363_SC-70-6, symbol Transistor_BJT:UMH3N
- added R1, R2, R8: 4.7k, Resistor_THT:R_Axial_DIN0207_L6.3mm_D2.5mm_P10.16mm_Horizontal, symbol PCM_SL_Resistors:10k
- added R3, R4, R5: 330R, Resistor_THT:R_Axial_DIN0207_L6.3mm_D2.5mm_P10.16mm_Horizontal, symbol PCM_SL_Resistors:1M
- added R6, R7: 10k, Resistor_THT:R_Axial_DIN0207_L6.3mm_D2.5mm_P10.16mm_Horizontal, symbol PCM_SL_Resistors:10k
- added SW1: RESET, Button_Switch_THT:SW_PUSH_6mm, symbol PCM_SL_Devices:Push_Button
- added SW2: FLASH, Button_Switch_THT:SW_PUSH_6mm, symbol PCM_SL_Devices:Push_Button
- added U1: AMS1117-3.3, Package_TO_SOT_SMD:SOT-223-3_TabPin2, symbol Regulator_Linear:AMS1117-3.3
- added U2: CH340C, Package_SO:SOIC-16_3.9x9.9mm_P1.27mm, symbol Interface_USB:CH340C
- added U3: ESP32-WROOM, SparkFun-RF:ESP32-WROOM-32D-DFM_PASTE, symbol SparkFun-RF:ESP32-WROOM
- added U4: PCA9555D, Package_SO:SOIC-24W_7.5x15.4mm_P1.27mm, symbol Interface_Expansion:PCA9555D
- added Y1: 12MHz, Crystal:Crystal_HC49-4H_Vertical, symbol PCM_SL_Devices:Crystal_16MHz
Connections:
- new net: Q1.7 (IN7), U4.10 (IO0_6)
- new net: Q1.8 (IN8), U4.11 (IO0_7)
- new net: Q2.1 (IN1), U4.13 (IO1_0)
- new net: Q2.2 (IN2), U4.14 (IO1_1)
- new net: Q2.3 (IN3), U4.15 (IO1_2)
- new net: Q2.4 (IN4), U4.16 (IO1_3)
- new net: Q1.1 (IN1), U4.4 (IO0_0)
- new net: Q1.2 (IN2), U4.5 (IO0_1)
- new net: Q1.3 (IN3), U4.6 (IO0_2)
- new net: Q1.4 (IN4), U4.7 (IO0_3)
- new net: Q1.5 (IN5), U4.8 (IO0_4)
- new net: Q1.6 (IN6), U4.9 (IO0_5)
- new net: C1.1, C2.1, C3.2, D5.1 (K), J1.4 (Pin_4), U1.3 (VI)
- new net: K1.11A, K1.11B, K2.11A, K2.11B
- new net: K3.11A, K3.11B, K4.11A, K4.11B
- new net: J3.1, K4.14
- new net: D3.2 (A), R4.2
- new net: C4.1, D1.2 (A), U1.2 (VO)
- new net: J5.1, K10.14
- new net: K10.11A, K10.11B, K7.11A, K7.11B
- new net: D4.2 (A), R5.2
- new net: K11.11A, K11.11B, K8.11A, K8.11B
- new net: J6.1, K11.14
- new net: J7.1, K12.14
- new net: J4.1, K6.14
- new net: K5.11A, K5.11B, K6.11A, K6.11B
- new net: J2.1, K1.14
- new net: C9.1, U2.7 (Xi), Y1.2
- new net: D2.2 (A), R3.2
- new net: C8.1, U2.8 (Xo), Y1.1
- new net: C5.2, JP1.1 (A), U2.4 (V3)
- new net: J1.2 (Pin_2), U2.5 (UD+)
- new net: J1.3 (Pin_3), U2.6 (UD-)
- new net: K12.11A, K12.11B, K9.11A, K9.11B
- new net +12V: C10.1, C11.1, D10.1 (K), D11.1 (K), D12.1 (K), D13.1 (K), D14.1 (K), D15.1 (K), D16.1 (K), D17.1 (K), D6.1 (K), D7.1 (K), D8.1 (K), D9.1 (K), K1.A2, K10.A2, K11.A2, K12.A2, K2.A1, K3.A1, K4.A2, K5.A1, K6.A2, K7.A1, K8.A1, K9.A1, Q1.10 (COM), Q2.10 (COM)
- new net +3.3V: C12.1, C7.2, D1.1 (K), D18.1 (K), JP1.2 (B), R1.2, R2.2, R3.1, R4.1, R6.2, R7.2, R8.2, U2.16 (VCC), U3.2 (VDD), U4.24 (VDD)
- new net DTR: Q3.2 (B1), Q3.4 (E2), U2.13 (~{DTR})
- new net EN: C6.2, Q3.6 (C1), R6.1, SW1.2, U3.3 (EN)
- new net GND: C1.2, C10.2, C11.2, C12.2, C2.2, C3.1, C4.2, C5.1, C6.1, C7.1, C8.2, C9.2, D18.2 (A), D4.1 (K), D5.2 (A), J1.1 (Pin_1), Q1.9 (GND), Q2.9 (GND), SW1.1, SW2.1, U1.1 (GND), U2.1 (GND), U3.1 (GND), U3.15 (GND), U3.38 (GND), U3.49.1 (GND), U3.49.2 (GND), U3.49.3 (GND), U3.49.4 (GND), U3.49.5 (GND), U3.49.6 (GND), U3.49.7 (GND), U3.49.8 (GND), U3.49.9 (GND), U4.12 (VSS), U4.2 (A1), U4.21 (A0), U4.3 (A2)
- new net GPIO0: Q3.3 (C2), R7.1, SW2.2, U3.25 (IOA0)
- new net GPIO12: U3.14 (IOA12)
- new net GPIO13: U3.16 (IOA13)
- new net GPIO14: U3.13 (IOA14)
- new net GPIO15: U3.23 (IOA15)
- new net GPIO16: U3.27 (IO16)
- new net GPIO17: U3.28 (IO17)
- new net GPIO18/SCK: U3.30 (IO18)
- new net GPIO19/MISO: U3.31 (IO19)
- new net GPIO1/TX: D2.1 (K), U2.3 (RXD), U3.35 (TXD0/IO1)
- new net GPIO2: R5.1, U3.24 (IOA2)
- new net GPIO21/SDA: R2.1, U3.33 (IO21), U4.23 (SDA)
- new net GPIO22/SCL: R1.1, U3.36 (IO22), U4.22 (SCL)
- new net GPIO23/MOSI: U3.37 (IO23)
- new net GPIO25: U3.10 (IOA25)
- new net GPIO26: U3.11 (IOA26)
- new net GPIO27: U3.12 (IOA27)
- new net GPIO32: U3.8 (IOA32)
- new net GPIO33: U3.9 (IOA33)
- new net GPIO34: U3.6 (IA34)
- new net GPIO35: U3.7 (IA35)
- new net GPIO36: U3.4 (IA36)
- new net GPIO39: U3.5 (IA39)
- new net GPIO3/RX: D3.1 (K), U2.2 (TXD), U3.34 (RXD0/IO3)
- new net GPIO4: U3.26 (IOA4)
- new net GPIO5/CS: U3.29 (IO5)
- new net IND_LED: U4.17 (IO1_4)
- new net INVERTER: K2.12, K3.12, K5.12, K7.12, K8.12, K9.12
- new net N: J2.2, J3.2, J4.2, J5.2, J6.2, J7.2
- new net NEPA: K2.14, K3.14, K5.14, K7.14, K8.14, K9.14
- new net RD1C1: D6.2 (A), K1.A1, Q1.18 (OUT1)
- new net RD1C2: D7.2 (A), K2.A2, Q1.17 (OUT2)
- new net RD1C3: D9.2 (A), K4.A1, Q1.16 (OUT3)
- new net RD1C4: D8.2 (A), K3.A2, Q1.15 (OUT4)
- new net RD1C5: D11.2 (A), K6.A1, Q1.14 (OUT5)
- new net RD1C6: D10.2 (A), K5.A2, Q1.13 (OUT6)
- new net RD1C7: D15.2 (A), K10.A1, Q1.12 (OUT7)
- new net RD1C8: D12.2 (A), K7.A2, Q1.11 (OUT8)
- new net RD2C1: D16.2 (A), K11.A1, Q2.18 (OUT1)
- new net RD2C2: D13.2 (A), K8.A2, Q2.17 (OUT2)
- new net RD2C3: D17.2 (A), K12.A1, Q2.16 (OUT3)
- new net RD2C4: D14.2 (A), K9.A2, Q2.15 (OUT4)
- new net RD2C5: Q2.14 (OUT5)
- new net RD2C6: Q2.13 (OUT6)
- new net RD2C7: Q2.12 (OUT7)
- new net RD2C8: Q2.11 (OUT8)
- new net RD_EN: U4.18 (IO1_5)
- new net RTS: Q3.1 (E1), Q3.5 (B2), U2.14 (~{RTS})
- new net S1_IN: U4.19 (IO1_6)
- new net S2_IN: U4.20 (IO1_7)
- new net ~{INT}: R8.1, U4.1 (~{INT})
- no-connect marks 0 -> 4
Other:
- note added: "CONTROL & COMMAND"
- note added: "DEBUGGING & PROGRAMMING"
- note added: "GPIO EXPANDER & RELAY DRIVER"
- note added: "If CH340G is used"
- note added: "LCD SCREEN & ROTARY ENCODER"
- note added: "POWER SUPPLY"
- note added: "RELAY & LOAD TERMINAL"

Commit message: update from home
Parts:
- added J9: 128X64 GLCD, symbol Connector:Screw_Terminal_01x20
- added R16, R9: 10K, Resistor_THT:R_Axial_DIN0207_L6.3mm_D2.5mm_P10.16mm_Horizontal, symbol Device:R_Small
- added RV2: 10K, symbol Device:R_Potentiometer_Small
- added SW3: RotaryEncoder_Switch, Rotary_Encoder:RotaryEncoder_Alps_EC12E-Switch_Vertical_H20mm, symbol Device:RotaryEncoder_Switch
Connections:
- net +3.3V: now also J9.19 (Pin_19)
- net GND: now also J9.1 (Pin_1), J9.15 (Pin_15), J9.20 (Pin_20), RV2.1, SW3.C, SW3.S2
- net GPIO18/SCK: now also J9.4 (Pin_4)
- net GPIO23/MOSI: now also J9.5 (Pin_5)
- net GPIO5/CS: now also J9.6 (Pin_6)
- new net: R16.1, SW3.A
- new net: J9.3 (Pin_3), RV2.2
- new net: R9.1, SW3.B
- new net +5V: J9.2 (Pin_2), R16.2, R9.2, RV2.3
Other:
- note added: "GRAPHIC LIQUID CRYSTAL DISPLAY"

Commit message: update from work(Schematic done)
Parts:
- removed R16, R9: 10K, Resistor_THT:R_Axial_DIN0207_L6.3mm_D2.5mm_P10.16mm_Horizontal, symbol Device:R_Small
- removed SW3: RotaryEncoder_Switch, Rotary_Encoder:RotaryEncoder_Alps_EC12E-Switch_Vertical_H20mm, symbol Device:RotaryEncoder_Switch
- added C13, C15, C17: 680uF_35V, Capacitor_THT:CP_Radial_D10.0mm_P5.00mm, symbol PCM_SL_Capacitors:470uF_35V
- added C14, C16, C18: 220uF_16V, Capacitor_THT:CP_Radial_D10.0mm_P5.00mm, symbol PCM_SL_Capacitors:470uF_35V
- added C19, C21: 2200uF/35V, Capacitor_THT:CP_Radial_D5.0mm_P2.00mm, symbol PCM_SL_Capacitors:4.7uF_16V
- added C20, C22: 100nF, symbol Device:C_Small
- added C23: 145J400V, symbol Device:C_Small
- added C24: 470uF/25V, Capacitor_THT:CP_Radial_D5.0mm_P2.00mm, symbol PCM_SL_Capacitors:4.7uF_16V
- added D19, D20, D21: 1N5824, Diode_THT:D_DO-201AD_P15.24mm_Horizontal, symbol Diode:1N5822
- added D22, D23: GBU8M, Diode_THT:Diode_Bridge_Vishay_GBU, symbol Diode_Bridge:GBU8M
- added D24, D25, D26, D27, D28: SM4001, Diode_SMD:D_MELF, symbol Diode:SM4001
- added D29: Blue, SparkFun-LED:LED_0603_1608Metric_Red, symbol SparkFun-LED:LED_Red_0603
- added DZ1: CMZ12, PCM_Diode_SMD_AKL:D_SOD-128, symbol PCM_Diode_Zener_AKL:CMZ12
- added J10: PZEM_LOAD, symbol Connector:Screw_Terminal_01x04
- added J11: CT, TerminalBlock_Phoenix:TerminalBlock_Phoenix_PT-1,5-2-5.0-H_1x02_P5.00mm_Horizontal, symbol PCM_SL_Screw_Terminal:Screw_Terminal_2_P5.00mm
- added J8: PZEM_SIG, symbol Connector:Screw_Terminal_01x04
- added JP2, JP3: ~, SparkFun-Jumper:Jumper_3_NO, symbol SparkFun-Jumper:SolderJumper_3_Open
- added K13: 10A RELAY, Relay_THT:Relay_SPDT_Finder_36.11, symbol Relay:FINDER-36.11
- added L1, L2, L3: 33uH, symbol Device:L_Small
- added OC1, OC2: PC817XFP, PCM_Package_DIP_AKL:SMDIP-4_W11.48mm, symbol PCM_Optocoupler_AKL:PC817XFP
- added Q4: UMH3N, Package_TO_SOT_SMD:SOT-363_SC-70-6, symbol Transistor_BJT:UMH3N
- added R10, R9: 10k, Resistor_THT:R_Axial_DIN0207_L6.3mm_D2.5mm_P10.16mm_Horizontal, symbol PCM_SL_Resistors:10k
- added R11: 150R, Resistor_THT:R_Axial_DIN0207_L6.3mm_D2.5mm_P10.16mm_Horizontal, symbol PCM_SL_Resistors:10k
- added R12, R14, R16: 680k, Resistor_THT:R_Axial_DIN0207_L6.3mm_D2.5mm_P10.16mm_Horizontal, symbol PCM_SL_Resistors:10k
- added R13, R15, R17: 6.8k, Resistor_THT:R_Axial_DIN0207_L6.3mm_D2.5mm_P10.16mm_Horizontal, symbol PCM_SL_Resistors:10k
- added R18, R21: 330R, Resistor_THT:R_Axial_DIN0207_L6.3mm_D2.5mm_P10.16mm_Horizontal, symbol PCM_SL_Resistors:1M
- added R19: 1M, Resistor_THT:R_Axial_DIN0207_L6.3mm_D2.5mm_P10.16mm_Horizontal, symbol PCM_SL_Resistors:10k
- added R20: 330R/2W, Resistor_THT:R_Axial_DIN0207_L6.3mm_D2.5mm_P10.16mm_Horizontal, symbol PCM_SL_Resistors:1M
- added R22: 100k, Resistor_THT:R_Axial_DIN0207_L6.3mm_D2.5mm_P10.16mm_Horizontal, symbol PCM_SL_Resistors:10k
- added SW4: RotaryEncoder, symbol Device:RotaryEncoder_Switch_MP
- added T1, T2: 2220-12V, symbol Device:Transformer_1P_1S
- added TP1, TP2, TP3, TP4, TP5, TP6, TP7, TP8, TP9: TestPoint, TestPoint:TestPoint_Pad_D1.5mm, symbol PCM_4ms_Connector:TestPoint
- added U5: LM2596S-3.3V, Package_TO_SOT_SMD:TO-263-5_TabPin3, symbol Regulator_Switching:LM2596S-3.3
- added U6: LM2596S-5V, Package_TO_SOT_SMD:TO-263-5_TabPin3, symbol Regulator_Switching:LM2596S-5
- added U7: LM2596S-12, Package_TO_SOT_SMD:TO-263-5_TabPin3, symbol Regulator_Switching:LM2596S-12
- D4: value Red -> GREEN
- K1, K10, K11, K12, K2, K3, K4, K5, K6, K7, K8, K9: value RAYEX-L90 -> 30A RELAY
- R1, R2, R8: value 4.7k -> 10k
Connections:
- net +12V: now also C18.1, L3.2, TP3.1, U7.4 (FB)
- net +3.3V: now also C14.1, L1.2, R10.2, R9.1, TP2.1, U5.4 (FB)
- net +5V: now also C16.1, J8.1 (Pin_1), L2.2, TP1.1, U6.4 (FB)
- net GND: now also C13.2, C14.2, C15.2, C16.2, C17.2, C18.2, C19.2, C20.1, C21.2, C22.1, D19.2 (A), D20.2 (A), D21.2 (A), D22.4 (-), D23.4 (-), D29.1 (K), J8.4 (Pin_4), OC1.2, OC1.3, OC2.3, SW4.C, SW4.MP, SW4.S2, U5.3 (GND), U5.5 (~{ON}/OFF), U6.3 (GND), U6.5 (~{ON}/OFF), U7.3 (GND)
- net GPIO16: now also JP3.1 (A)
- net GPIO17: now also JP2.3 (C)
- net GPIO1/TX: now also JP2.1 (A)
- net GPIO25: now also R9.2, SW4.A
- net GPIO26: now also R10.1, SW4.B
- net GPIO27: now also SW4.S1
- net GPIO3/RX: now also JP3.3 (C)
- net IND_LED: now also R21.1
- net INVERTER: now also K13.12, R12.2
- net N: now also J10.2 (Pin_2), OC2.2, Q4.4 (E2), R13.1, R15.1, R17.1, R20.1, T1.2 (AB), T2.2 (AB)
- net NEPA: now also C23.2, J10.1 (Pin_1), K13.14, R14.2, R16.2, R19.2
- net at C1.1, C2.1, C3.2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: now also TP6.1
- net at C4.1, D1.2 (A), U1.2 (VO): now also TP5.1
- net RD_EN: no longer names the net of U4.18 (IO1_5)
- net RD_EN: now also R11.2
- net S1_IN renamed INVERTER_SENSE
- net INVERTER_SENSE: now also Q4.5 (B2), R12.1, R13.2, TP9.1
- net S2_IN renamed NEPA_SENSE
- net NEPA_SENSE: now also Q4.2 (B1), R16.1, R17.2, TP8.1
- new net: K13.11, T1.1 (AA), T2.1 (AA)
- new net: D24.2 (A), K13.A1, OC2.4
- new net: D21.1 (K), L3.1, U7.2 (OUT)
- new net: J8.2 (Pin_2), JP2.2 (B)
- new net: J8.3 (Pin_3), JP3.2 (B)
- new net: Q4.1 (E1), Q4.3 (C2), R18.1
- new net: Q4.6 (C1), R14.1, R15.2
- new net: D20.1 (K), L2.1, U6.2 (OUT)
- new net: C24.2, D25.2 (A), D26.2 (A), DZ1.2 (A)
- new net: OC1.4, R22.1, TP7.1, U7.5 (~{ON}/OFF)
- new net: D19.1 (K), L1.1, U5.2 (OUT)
- new net: C23.1, D25.1 (K), D27.2 (A), R19.1
- new net: OC2.1, R18.2
- new net: D26.1 (K), D28.2 (A), R20.2
- new net: D22.2, T2.3 (SA)
- new net: D22.3, T2.4 (SB)
- new net: D29.2 (A), R21.2
- new net: D23.2, T1.3 (SA)
- new net: D23.3, T1.4 (SB)
- new net 12V_EN: OC1.1, R11.1
- new net CT +: J10.4 (Pin_4), J11.2
- new net CT -: J10.3 (Pin_3), J11.1
- new net VCC1: C13.1, C15.1, C21.1, C22.2, D22.1 (+), U5.1 (VIN), U6.1 (VIN)
- new net VCC2: C17.1, C19.1, C20.2, D23.1 (+), R22.2, U7.1 (VIN)
- new net VCC3: C24.1, D24.1 (K), D27.1 (K), D28.1 (K), DZ1.1 (K), K13.A2, TP4.1
- no-connect marks 4 -> 37
Other:
- note added: "100A"
- note added: "LCD SCREEN"
- note added: "POWER SENSOR"
- note added: "PZEM004T"
- note added: "ROTARY ENCODER"
- note added: "VOLTAGE REGULATORS"
- note removed: "LCD SCREEN & ROTARY ENCODER"
- company: (none) -> JSITECH
- title: (none) -> SMART HOME ENERGY MANAGEMENT SYSTEM
- moved on the sheet: C1, C10, C11, C12, C2, C3, C4, C5, C6, C7, C8, C9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

Commit message: update
Parts:
- C1: renamed from C17; footprint Capacitor_THT:CP_Radial_D10.0mm_P5.00mm -> Capacitor_SMD:CP_Elec_10x12.5
- C10: renamed from C19; footprint Capacitor_THT:CP_Radial_D5.0mm_P2.00mm -> Capacitor_THT:CP_Radial_D18.0mm_P7.50mm
- C11: renamed from C16; footprint Capacitor_THT:CP_Radial_D10.0mm_P5.00mm -> Capacitor_SMD:CP_Elec_6.3x7.7
- C12: renamed from C22; footprint (none) -> Capacitor_SMD:C_0805_2012Metric
- C13: renamed from C20; footprint (none) -> Capacitor_SMD:C_0805_2012Metric
- C14: renamed from C24; footprint Capacitor_THT:CP_Radial_D5.0mm_P2.00mm -> Capacitor_SMD:CP_Elec_8x11.9
- C15: renamed from C1; footprint Capacitor_THT:CP_Radial_D5.0mm_P2.00mm -> Capacitor_Tantalum_SMD:CP_EIA-3216-18_Kemet-A
- C16: renamed from C2; footprint Capacitor_THT:CP_Radial_D5.0mm_P2.00mm -> Capacitor_Tantalum_SMD:CP_EIA-3216-18_Kemet-A
- C18: renamed from C3; footprint (none) -> Capacitor_SMD:C_0805_2012Metric
- C19: renamed from C4; footprint Capacitor_THT:CP_Radial_D5.0mm_P2.00mm -> Capacitor_Tantalum_SMD:CP_EIA-3216-18_Kemet-A
- C2: renamed from C13; footprint Capacitor_THT:CP_Radial_D10.0mm_P5.00mm -> Capacitor_SMD:CP_Elec_10x12.5
- C20: renamed from C9; footprint (none) -> Capacitor_SMD:C_0603_1608Metric
- C21: renamed from C8; footprint (none) -> Capacitor_SMD:C_0603_1608Metric
- C22: renamed from C5; footprint (none) -> Capacitor_SMD:C_0805_2012Metric
- C23: renamed from C10; value 0.1uF/25V -> 100nF
- C24: renamed from C11; value 0.1uF/25V -> 100nF
- C3: renamed from C6; footprint Capacitor_THT:C_Disc_D5.0mm_W2.5mm_P2.50mm -> Capacitor_SMD:C_0805_2012Metric
- C4: renamed from C7; footprint Capacitor_THT:C_Disc_D5.0mm_W2.5mm_P2.50mm -> Capacitor_SMD:C_0805_2012Metric
- C5: renamed from C14; footprint Capacitor_THT:CP_Radial_D10.0mm_P5.00mm -> Capacitor_SMD:CP_Elec_6.3x7.7
- C6: renamed from C18; footprint Capacitor_THT:CP_Radial_D10.0mm_P5.00mm -> Capacitor_SMD:CP_Elec_6.3x7.7
- C7: renamed from C15; footprint Capacitor_THT:CP_Radial_D10.0mm_P5.00mm -> Capacitor_SMD:CP_Elec_10x12.5
- C9: renamed from C21; footprint Capacitor_THT:CP_Radial_D5.0mm_P2.00mm -> Capacitor_THT:CP_Radial_D18.0mm_P7.50mm
- D1: renamed from D29; footprint SparkFun-LED:LED_0603_1608Metric_Red -> LED_SMD:LED_0805_2012Metric
- D10: renamed from D27; footprint Diode_SMD:D_MELF -> Diode_SMD:D_SMA
- D11: renamed from D28; footprint Diode_SMD:D_MELF -> Diode_SMD:D_SMA
- D12: renamed from D20; footprint Diode_THT:D_DO-201AD_P15.24mm_Horizontal -> Diode_SMD:D_SMA
- D15: renamed from D18; footprint Diode_SMD:D_MELF -> Diode_SMD:D_SMA
- D18: renamed from D7; footprint Diode_SMD:D_MELF -> Diode_SMD:D_SMA
- D19: renamed from D8; footprint Diode_SMD:D_MELF -> Diode_SMD:D_SMA
- D2: renamed from D19; footprint Diode_THT:D_DO-201AD_P15.24mm_Horizontal -> Diode_SMD:D_SMA
- D20: renamed from D10; footprint Diode_SMD:D_MELF -> Diode_SMD:D_SMA
- D21: renamed from D12; footprint Diode_SMD:D_MELF -> Diode_SMD:D_SMA
- D22: renamed from D13; footprint Diode_SMD:D_MELF -> Diode_SMD:D_SMA
- D23: renamed from D14; footprint Diode_SMD:D_MELF -> Diode_SMD:D_SMA
- D24: renamed from D6; footprint Diode_SMD:D_MELF -> Diode_SMD:D_SMA
- D25: renamed from D9; footprint Diode_SMD:D_MELF -> Diode_SMD:D_SMA
- D26: renamed from D11; footprint Diode_SMD:D_MELF -> Diode_SMD:D_SMA
- D27: renamed from D15; footprint Diode_SMD:D_MELF -> Diode_SMD:D_SMA
- D28: renamed from D16; footprint Diode_SMD:D_MELF -> Diode_SMD:D_SMA
- D29: renamed from D17; footprint Diode_SMD:D_MELF -> Diode_SMD:D_SMA
- D3: renamed from D21; footprint Diode_THT:D_DO-201AD_P15.24mm_Horizontal -> Diode_SMD:D_SMA
- D5: renamed from D24; footprint Diode_SMD:D_MELF -> Diode_SMD:D_SMA
- D6: renamed from D25; footprint Diode_SMD:D_MELF -> Diode_SMD:D_SMA
- D7: renamed from D26; footprint Diode_SMD:D_MELF -> Diode_SMD:D_SMA
- renumbered C12 to C17, C23 to C8, D5 to D13, D1 to D14, D2 to D16, D3 to D17, D22 to D8, D23 to D9, J11 to J1, J6 to J10, J7 to J11, J10 to J2, J8 to J3, J1 to J4, J9 to J5, J2 to J6, J3 to J7, J4 to J8, J5 to J9, JP2 to JP1, JP3 to JP2, JP1 to JP3, K13 to K1, K6 to K10, K10 to K11, K11 to K12, K12 to K13, K5 to K4, K7 to K5, K8 to K6, K9 to K7, K1 to K8, K4 to K9, L3 to L2, L2 to L3, Q4 to Q1, Q3 to Q2, Q1 to Q3, Q2 to Q4, R16 to R1, R6 to R10, R5 to R11, R7 to R12, R19 to R13, R20 to R14, R2 to R15, R1 to R16, R8 to R17, R11 to R18, R3 to R19, R12 to R2, R4 to R20, R10 to R21, R9 to R22, R22 to R3, R13 to R4, R17 to R5, R21 to R6, R14 to R7, R15 to R8, R18 to R9, RV2 to RV1, SW4 to SW3, T2 to T1, T1 to T2, TP8 to TP1, TP9 to TP2, TP7 to TP3, TP2 to TP4, TP3 to TP5, TP1 to TP6, TP4 to TP7, TP6 to TP8, TP5 to TP9, U5 to U1, U7 to U2, U6 to U4, U1 to U5, U4 to U6, U2 to U7
