File: ESP32/Smart Home Energy Management System/Smart Home Energy Management System.kicad_sch (KiCad schematic)
At the start: 149 parts, among them J1 CT, J10 LOAD 3, J11 LOAD 2, J12 DISPLAY, J13 TRANS-IN, J14 TRANS 2-OUT, J15 TRANS 1-OUT, J16 N, J17 N, J18 N, J19 N, J2 PZEM_LOAD, J20 N, J21 N, J22 N, J23 N, J24 LOAD 1, J25 NEPA, J3 PZEM_SIG, J4 USB_C Conn, J5 128X64 GLCD, J6 INVERTER, J7 LOAD 6, J8 LOAD 5, J9 LOAD 4, K1 10A RELAY, K10 30A RELAY, K11 30A RELAY, K12 30A RELAY, K13 30A RELAY, K2 30A RELAY, K3 30A RELAY, K4 30A RELAY, K5 30A RELAY, K6 30A RELAY, K7 30A RELAY, K8 30A RELAY, K9 30A RELAY, Q1 UMH3N, Q2 UMH3N, Q3 ULN2803ADWR, Q4 ULN2803ADWR, SW1 RESET, SW2 FLASH, SW3 RotaryEncoder, T1 2220-12V, T2 2220-12V, U1 LM2596S-3.3V, U2 LM2596S-12, U3 ESP32-WROOM, U4 LM2596S-5V, U5 AMS1117-3.3, U6 PCA9555D, U7 CH340C, Y1 12MHz

Commit message: update from home
Parts:
- J7: footprint (none) -> TestPoint:TestPoint_Plated_Hole_D5.0mm
Changed lines of the file:
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@@
 			)
 		)
-		(property "Footprint" ""
+		(property "Footprint" "TestPoint:TestPoint_Plated_Hole_D5.0mm"
 			(at 386.08 48.26 0)
 			(effects

Commit message: update from work
Parts:
- added TP10, TP11, TP12, TP13, TP14, TP15, TP16, TP17: TestPoint, TestPoint:TestPoint_Pad_D1.5mm, symbol PCM_4ms_Connector:TestPoint
- D1, D16, D17, D4: footprint PCM_JLCPCB:LED-SMD_4P-L1.6-W1.5_XL-1615RGBC-WS2812B -> LED_THT:LED_D3.0mm
- J10, J11, J16, J17, J18, J19, J20, J21, J22, J23, J24, J25, J6, J8, J9: footprint (none) -> TestPoint:TestPoint_Plated_Hole_D5.0mm
- RV1: footprint PCM_JLCPCB:R_0805 -> Potentiometer_THT:Potentiometer_Bourns_3296W_Vertical
Connections:
- net EN: now also TP10.1
- net GND: now also C14.2, D6.2 (A), D7.2 (A), DZ1.2 (A), U1.6 (GND), U2.6 (GND), U3.39 (GND), U4.6 (GND), TP12.1, TP13.1; no longer U3.49.1 (GND), U3.49.2 (GND), U3.49.3 (GND), U3.49.4 (GND), U3.49.5 (GND), U3.49.6 (GND), U3.49.7 (GND), U3.49.8 (GND), U3.49.9 (GND)
- net GPIO0: now also TP11.1
- net GPIO1/TX: now also TP16.1
- net GPIO21/SDA: now also TP15.1
- net GPIO22/SCL: now also TP14.1
- net GPIO3/RX: now also TP17.1
- net at C19.1, D14.2 (A), TP9.1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: now also U5.4 (VO)

Commit message: update from work
Parts:
- removed D15: SM4001, PCM_JLCPCB:D_SMA, symbol Diode:SM4001
- added C25: 100nF, PCM_JLCPCB:C_0805, symbol PCM_SL_Capacitors:104_Ceramic
- renumbered J25 to J1, J17 to J10, J3 to J11, J18 to J12, J19 to J13, J4 to J14, J5 to J16, J13 to J17, J14 to J18, J12 to J19, J6 to J2, J7 to J20, J8 to J21, J9 to J22, J10 to J23, J11 to J24, J24 to J25, J1 to J3, J20 to J4, J21 to J5, J2 to J6, J22 to J7, J23 to J8, J16 to J9, TP13 to TP1, TP5 to TP10, TP12 to TP11, TP6 to TP12, TP7 to TP13, TP8 to TP16, TP9 to TP17, TP1 to TP2, TP2 to TP3, TP3 to TP4, TP10 to TP5, TP11 to TP6, TP16 to TP7, TP17 to TP8, TP4 to TP9
Connections:
- net +3.3V: now also C25.2
- net GND: now also C25.1

Commit message: update from work
Parts:
- removed J12, J13, J4, J5, J7, J8: N, TestPoint:TestPoint_Plated_Hole_D5.0mm, symbol Connector:Screw_Terminal_01x01
Connections:
- net SELECT6: now reaches K2.11A, K2.11B, K8.11A, K8.11B
- net SELECT5: now reaches K3.11A, K3.11B, K9.11A, K9.11B
- net LOAD5: now reaches J21.1 (Pin_1), K9.14
- net LOAD2: now reaches J24.1 (Pin_1), K12.14
- net SELECT3: now reaches K11.11A, K11.11B, K5.11A, K5.11B
- net SELECT2: now reaches K12.11A, K12.11B, K6.11A, K6.11B
- net SELECT4: now reaches K10.11A, K10.11B, K4.11A, K4.11B
- net LOAD4: now reaches J22.1 (Pin_1), K10.14
- net LOAD3: now reaches J23.1 (Pin_1), K11.14
- net SELECT1: now reaches K13.11A, K13.11B, K7.11A, K7.11B
- net LOAD1: now reaches J25.1 (Pin_1), K13.14
- net LOAD6: now reaches J20.1 (Pin_1), K8.14

Commit message: update from work
Parts:
- removed J9: N, TestPoint:TestPoint_Plated_Hole_D5.0mm, symbol Connector:Screw_Terminal_01x01
Connections:
- net TXP: now reaches J11.2 (Pin_2), JP1.2 (B)
- net RXN: now reaches J11.3 (Pin_3), JP2.2 (B)
Changed lines of the file:
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@@
 	)
 	(junction
-		(at 64.77 266.7)
-		(diameter 0)
-		(color 0 0 0 0)
-	)
-	(junction
 		(at 242.57 91.44)
 		(diameter 0)
@@
 	(wire
 		(pts
-			(xy 64.77 266.7) (xy 64.77 269.24)
-		)
-		(stroke
-			(width 0)
-			(type default)
-		)
-	)
-	(wire
-		(pts
 			(xy 74.93 48.26) (xy 74.93 49.53)
 		)
@@
 	(wire
 		(pts
-			(xy 60.96 266.7) (xy 64.77 266.7)
+			(xy 66.04 266.7) (xy 69.85 266.7)
 		)
 		(stroke
@@
 	(wire
 		(pts
-			(xy 64.77 266.7) (xy 69.85 266.7)
-		)
-		(stroke
-			(width 0)
-			(type default)
-		)
-	)
-	(wire
-		(pts
 			(xy 250.19 132.08) (xy 247.65 132.08)
 		)
@@
 		)
 	)
+	(label "RXN"
+		(at 107.95 158.75 0)
+		(effects
+			(font
+				(size 1.27 1.27)
+			)
+			(justify left bottom)
+		)
+		(property "Netclass" "DIFF"
+			(at 102.616 157.988 0)
+			(effects
+				(font
+					(size 1.27 1.27)
+					(italic yes)
+				)
+				(justify left)
+			)
+		)
+	)
 	(label "INVERTER"
 		(at 300.99 80.01 0)
@@
 	)
 	(label "N"
-		(at 60.96 266.7 0)
+		(at 66.04 266.7 0)
 		(effects
 			(font
@@
 		)
 	)
+	(label "TXP"
+		(at 107.95 156.21 0)
+		(effects
+			(font
+				(size 1.27 1.27)
+			)
+			(justify left bottom)
+		)
+		(property "Netclass" "DIFF"
+			(at 102.616 155.448 0)
+			(effects
+				(font
+					(size 1.27 1.27)
+					(italic yes)
+				)
+				(justify left)
+			)
+		)
+	)
 	(label "DTR"
 		(at 232.41 52.07 180)
@@
 					(unit 1)
 				)
-			)
-		)
-	)
-	(symbol
-		(lib_id "Connector:Screw_Terminal_01x01")
-		(at 64.77 274.32 270)
-		(unit 1)
-		(exclude_from_sim no)
-		(in_bom yes)
-		(on_board yes)
-		(dnp no)
-		(property "Reference" "J9"
-			(at 66.548 274.828 90)
-			(effects
-				(font
-					(size 1.27 1.27)
-				)
-				(justify left)
-				(hide yes)
-			)
-		)
-		(property "Value" "N"
-			(at 64.262 276.86 90)
-			(effects
-				(font
-					(size 1.27 1.27)
-				)
-				(justify left)
-			)
-		)
-		(property "Footprint" "TestPoint:TestPoint_Plated_Hole_D5.0mm"
-			(at 64.77 274.32 0)
-			(effects
-				(font
-					(size 1.27 1.27)
-				)
-				(hide yes)
-			)
-		)
-		(property "Datasheet" "~"
-			(at 64.77 274.32 0)
-			(effects
-				(font
-					(size 1.27 1.27)
-				)
-				(hide yes)
-			)
-		)
-		(property "Description" "Generic screw terminal, single row, 01x01, script generated (kicad-library-utils/schlib/autogen/connector/)"
-			(at 64.77 274.32 0)
-			(effects
-				(font
-					(size 1.27 1.27)
-				)
-				(hide yes)
-			)
-		)
-		(pin "1"
-		)
-		(instances
-			(project ""
-				(path "/e0de9594-c08d-4dbe-8d5b-5599e595edda"
-					(reference "J9")
-					(unit 1)
-				)

Commit message: update from work
Parts:
- added C26, C27: 10uF_16V, PCM_JLCPCB:C_CASE-B-3528-21(mm), symbol PCM_SL_Capacitors:10uF_16V
- added D15, D30: SM4007PL, PCM_JLCPCB:D_SMA, symbol Diode:SM4001
Connections:
- net INVERTER: now also D30.2 (A); no longer R2.2
- net INVERTER_SENSE: now also C27.1
- net N: now also C26.2, C27.2
- net NEPA: now also D15.2 (A); no longer R1.2
- net NEPA_SENSE: now also C26.1
- new net: D15.1 (K), R1.2
- new net: D30.1 (K), R2.2
Other:
- moved on the sheet: R1, R2, R4, TP3

Commit message: update from work
Changed lines of the file:
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@@
 	)
 	(junction
+		(at 130.81 27.94)
+		(diameter 0)
+		(color 0 0 0 0)
+	)
+	(junction
 		(at 229.87 66.04)
 		(diameter 0)
@@
 	)
 	(junction
+		(at 63.5 27.94)
+		(diameter 0)
+		(color 0 0 0 0)
+	)
+	(junction
 		(at 308.61 214.63)
 		(diameter 0)
@@
 	)
 	(junction
+		(at 73.66 54.61)
+		(diameter 0)
+		(color 0 0 0 0)
+	)
+	(junction
 		(at 82.55 49.53)
 		(diameter 0)
@@
 	(wire
 		(pts
+			(xy 73.66 45.72) (xy 73.66 54.61)
+		)
+		(stroke
+			(width 0)
+			(type default)
+		)
+	)
+	(wire
+		(pts
 			(xy 115.57 158.75) (xy 125.73 158.75)
 		)
@@
 	(wire
 		(pts
+			(xy 73.66 54.61) (xy 74.93 54.61)
+		)
+		(stroke
+			(width 0)
+			(type default)
+		)
+	)
+	(wire
+		(pts
 			(xy 129.54 38.1) (xy 129.54 39.37)
 		)
@@
 	(wire
 		(pts
+			(xy 63.5 27.94) (xy 64.77 27.94)
+		)
+		(stroke
+			(width 0)
+			(type default)
+		)
+	)
+	(wire
+		(pts
 			(xy 351.79 172.72) (xy 351.79 175.26)
 		)
@@
 	(wire
 		(pts
+			(xy 63.5 19.05) (xy 63.5 27.94)
+		)
+		(stroke
+			(width 0)
+			(type default)
+		)
+	)
+	(wire
+		(pts
 			(xy 351.79 175.26) (xy 359.41 175.26)
 		)
@@
 	(wire
 		(pts
-			(xy 62.23 27.94) (xy 64.77 27.94)
+			(xy 62.23 27.94) (xy 63.5 27.94)
 		)
 		(stroke
@@
 	(wire
 		(pts
+			(xy 130.81 27.94) (xy 132.08 27.94)
+		)
+		(stroke
+			(width 0)
+			(type default)
+		)
+	)
+	(wire
+		(pts
 			(xy 49.53 38.1) (xy 62.23 38.1)
 		)
@@
 	(wire
 		(pts
-			(xy 129.54 27.94) (xy 132.08 27.94)
+			(xy 129.54 27.94) (xy 130.81 27.94)
 		)
 		(stroke
@@
 	(wire
 		(pts
+			(xy 130.81 19.05) (xy 130.81 27.94)
+		)
+		(stroke
+			(width 0)
+			(type default)
+		)
+	)
+	(wire
+		(pts
 			(xy 45.72 57.15) (xy 45.72 54.61)
 		)
@@
 	(wire
 		(pts
-			(xy 72.39 54.61) (xy 74.93 54.61)
+			(xy 72.39 54.61) (xy 73.66 54.61)
 		)
 		(stroke
@@
 		(length 2.54)
 		(shape round)
+		(at 73.66 45.72 0)
+		(fields_autoplaced yes)
+		(effects
+			(font
+				(size 1.27 1.27)
+			)
+			(justify left bottom)
+		)
+		(property "Netclass" "PWR"
+			(at 74.2696 43.18 0)
+			(effects
+				(font
+					(size 1.27 1.27)
+				)
+				(justify left)
+			)
+		)
+		(property "Component Class" ""
+			(at -25.4 24.13 0)
+			(effects
+				(font
+					(size 1.27 1.27)
+					(italic yes)
+				)
+			)
+		)
+	)
+	(netclass_flag ""
+		(length 2.54)
+		(shape round)
 		(at 332.74 45.72 0)
 		(fields_autoplaced yes)
@@
 		(length 2.54)
 		(shape round)
+		(at 63.5 19.05 0)
+		(fields_autoplaced yes)
+		(effects
+			(font
+				(size 1.27 1.27)
+			)
+			(justify left bottom)
+		)
+		(property "Netclass" "PWR"
+			(at 64.1096 16.51 0)
+			(effects
+				(font
+					(size 1.27 1.27)
+				)
+				(justify left)
+			)
+		)
+		(property "Component Class" ""
+			(at -35.56 -2.54 0)
+			(effects
+				(font
+					(size 1.27 1.27)
+					(italic yes)
+				)
+			)
+		)
+	)
+	(netclass_flag ""
+		(length 2.54)
+		(shape round)
 		(at 190.5 59.69 0)
 		(fields_autoplaced yes)
@@
 			(effects
 				(font
+					(size 1.27 1.27)
+					(italic yes)
+				)
+			)
+		)
+	)
+	(netclass_flag ""
+		(length 2.54)
+		(shape round)
+		(at 130.81 19.05 0)
+		(fields_autoplaced yes)
+		(effects
+			(font
+				(size 1.27 1.27)
+			)
+			(justify left bottom)
+		)
+		(property "Netclass" "PWR"
+			(at 131.4196 16.51 0)
+			(effects
+				(font
+					(size 1.27 1.27)
+				)
+				(justify left)
+			)
+		)
+		(property "Component Class" ""
+			(at 31.75 -2.54 0)
+			(effects
+				(font
