File: ESP32/Smart Home Energy Management System/Smart Home Energy Management System SCHEMATIC ONLY.kicad_sch (KiCad schematic)
At the start: 149 parts, among them J1 CT, J10 LOAD 3, J11 LOAD 2, J12 DISPLAY, J13 TRANS-IN, J14 TRANS 2-OUT, J15 TRANS 1-OUT, J16 N, J17 N, J18 N, J19 N, J2 PZEM_LOAD, J20 N, J21 N, J22 N, J23 N, J24 LOAD 1, J25 NEPA, J3 PZEM_SIG, J4 USB_C Conn, J5 128X64 GLCD, J6 INVERTER, J7 LOAD 6, J8 LOAD 5, J9 LOAD 4, K1 10A RELAY, K10 30A RELAY, K11 30A RELAY, K12 30A RELAY, K13 30A RELAY, K2 30A RELAY, K3 30A RELAY, K4 30A RELAY, K5 30A RELAY, K6 30A RELAY, K7 30A RELAY, K8 30A RELAY, K9 30A RELAY, Q1 UMH3N, Q2 UMH3N, Q3 ULN2803ADWR, Q4 ULN2803ADWR, SW1 RESET, SW2 FLASH, SW3 RotaryEncoder, T1 2220-12V, T2 2220-12V, U1 LM2596S-3.3V, U2 LM2596S-12, U3 ESP32-WROOM, U4 LM2596S-5V, U5 AMS1117-3.3, U6 PCA9555D, U7 CH340C, Y1 12MHz

Commit message: update from home
Parts:
- removed J10: LOAD 3, symbol Connector:Screw_Terminal_01x01
- removed J11: LOAD 2, symbol Connector:Screw_Terminal_01x01
- removed J12: DISPLAY, Connector_PinHeader_2.54mm:PinHeader_1x12_P2.54mm_Vertical, symbol Connector:Screw_Terminal_01x12
- removed J13: TRANS-IN, TerminalBlock_Phoenix:TerminalBlock_Phoenix_PT-1,5-2-5.0-H_1x02_P5.00mm_Horizontal, symbol PCM_SL_Screw_Terminal:Screw_Terminal_2_P5.00mm
- removed J14: TRANS 2-OUT, TerminalBlock_Phoenix:TerminalBlock_Phoenix_PT-1,5-2-5.0-H_1x02_P5.00mm_Horizontal, symbol PCM_SL_Screw_Terminal:Screw_Terminal_2_P5.00mm
- removed J15: TRANS 1-OUT, TerminalBlock_Phoenix:TerminalBlock_Phoenix_PT-1,5-2-5.0-H_1x02_P5.00mm_Horizontal, symbol PCM_SL_Screw_Terminal:Screw_Terminal_2_P5.00mm
- removed J16, J17, J18, J19, J20, J21, J22, J23: N, symbol Connector:Screw_Terminal_01x01
- removed J24: LOAD 1, symbol Connector:Screw_Terminal_01x01
- removed J25: NEPA, symbol Connector:Screw_Terminal_01x01
- removed J6: INVERTER, symbol Connector:Screw_Terminal_01x01
- removed J7: LOAD 6, symbol Connector:Screw_Terminal_01x01
- removed J8: LOAD 5, symbol Connector:Screw_Terminal_01x01
- removed J9: LOAD 4, symbol Connector:Screw_Terminal_01x01
- added J10, J11, J6, J7, J8, J9: LOAD, TerminalBlock_Phoenix:TerminalBlock_Phoenix_PT-1,5-2-5.0-H_1x02_P5.00mm_Horizontal, symbol PCM_SL_Screw_Terminal:Screw_Terminal_2_P5.00mm
- C12, C13, C17, C18, C22, C23, C24, C3, C4: footprint PCM_JLCPCB:C_0805 -> Capacitor_SMD:C_0805_2012Metric
- C15, C16: footprint PCM_JLCPCB:C_CASE-B-3528-21(mm) -> Capacitor_Tantalum_SMD:CP_EIA-3216-18_Kemet-A
- C20, C21: footprint PCM_JLCPCB:C_0805 -> Capacitor_SMD:C_0603_1608Metric
- C8: footprint Capacitor_THT:C_Rect_L19.0mm_W6.0mm_P15.00mm_MKS4 -> (none)
- D1, D16, D17: footprint PCM_JLCPCB:LED-SMD_4P-L1.6-W1.5_XL-1615RGBC-WS2812B -> LED_SMD:LED_0805_2012Metric
- D10, D11, D12, D13, D14, D15, D18, D19, D2, D20, D21, D22, D23, D24, D25, D26, D27, D28, D29, D3, D5, D6, D7: footprint PCM_JLCPCB:D_SMA -> Diode_SMD:D_SMA
- D4: footprint PCM_JLCPCB:LED-SMD_4P-L1.6-W1.5_XL-1615RGBC-WS2812B -> SparkFun-LED:LED_0603_1608Metric_Red
- DZ1: footprint PCM_JLCPCB:D_SOD-123 -> PCM_Diode_SMD_AKL:D_SOD-128
- J2: footprint TerminalBlock:TerminalBlock_MaiXu_MX126-5.0-04P_1x04_P5.00mm -> (none)
- J3: footprint Connector_PinHeader_2.54mm:PinHeader_1x04_P2.54mm_Vertical -> (none)
- JP1, JP2: footprint Jumper:SolderJumper-3_P1.3mm_Open_Pad1.0x1.5mm -> SparkFun-Jumper:Jumper_3_NO
- JP3: footprint Jumper:SolderJumper-2_P1.3mm_Open_Pad1.0x1.5mm -> SparkFun-Jumper:Jumper_2_NO
- L1, L2, L3: footprint Inductor_SMD:L_12x12mm_H6mm -> (none)
- OC1, OC2: footprint PCM_JLCPCB:SOP-4_4.4x2.6mm_P1.27mm -> PCM_Package_DIP_AKL:SMDIP-4_W11.48mm
- Q1, Q2: footprint PCM_JLCPCB:SOT-363_SC-70-6 -> Package_TO_SOT_SMD:SOT-363_SC-70-6
- Q3, Q4: footprint digikey-footprints:SOIC-18_W7.5mm -> digikey-footprints:DIP-18_W7.62mm
- R1, R10, R11, R12, R15, R16, R17, R18, R19, R2, R20, R21, R22, R3, R4, R5, R6, R7, R8, R9: footprint PCM_JLCPCB:R_0805 -> Resistor_THT:R_Axial_DIN0207_L6.3mm_D2.5mm_P10.16mm_Horizontal
- R14: footprint Resistor_THT:R_Axial_DIN0309_L9.0mm_D3.2mm_P20.32mm_Horizontal -> Resistor_THT:R_Axial_DIN0207_L6.3mm_D2.5mm_P10.16mm_Horizontal
- RV1: footprint PCM_JLCPCB:R_0805 -> (none)
- SW1, SW2: footprint PCM_JLCPCB:SW_TS-1088-AR02016 -> Button_Switch_THT:SW_PUSH_6mm
- U1, U2, U4: footprint PCM_JLCPCB:TO-263-5_L10.2-W8.9-P1.70-TL -> Package_TO_SOT_SMD:TO-263-5_TabPin3
- U3: footprint RF_Module:ESP32-WROOM-32E -> SparkFun-RF:ESP32-WROOM-32D-DFM_PASTE
- U5: footprint PCM_JLCPCB:SOT-223-3_L6.5-W3.4-P2.30-LS7.0-BR -> Package_TO_SOT_SMD:SOT-223-3_TabPin2
- U7: footprint PCM_JLCPCB:SOIC-16_3.9x9.9mm_P1.27mm -> Package_SO:SOIC-16_3.9x9.9mm_P1.27mm
- Y1: footprint PCM_JLCPCB:CRYSTAL-SMD_L11.5-W4.8-LS12.7 -> Crystal:Crystal_HC49-4H_Vertical
Connections:
- net N: now also J10.2, J11.2, J6.2, J7.2, J8.2, J9.2
- net at K9.14: now also J7.1
- net at K12.14: now also J10.1
- net at K10.14: now also J8.1
- net at K11.14: now also J9.1
- net at K13.14: now also J11.1
- net at K8.14: now also J6.1
- net 1TR 1: no longer names the net of D8.3, T1.4 (SB)
- net 1TR 2: no longer names the net of D8.2, T1.3 (SA)
- net 2TR 1: no longer names the net of D9.3, T2.4 (SB)
- net 2TR 2: no longer names the net of D9.2, T2.3 (SA)
- net CONST: no longer names the net of J5.3 (Pin_3), RV1.2
- net TRANS-IN: no longer names the net of K1.11, T1.1 (AA), T2.1 (AA)
Other:
- moved on the sheet: RV1
