File: ESP32/Smart Home Energy Management System/Smart Home Energy Management System.kicad_pcb (KiCad board)
At the start: 2 copper layers, 2 parts, among them J13 PZEM MODULE, J6 PZEM TERMINAL

Commit message: update from work
Parts:
- added C1: 680uF_35V, Capacitor_SMD:CP_Elec_10x12.5, F.Cu at (26.6, 102.2)
- added C10: 2200uF/35V, Capacitor_THT:CP_Radial_D18.0mm_P7.50mm, F.Cu at (5.62, 125.5)
- added C11: 220uF_16V, Capacitor_SMD:CP_Elec_6.3x7.7, F.Cu at (34.3, 155.7)
- added C12: 100nF, PCM_JLCPCB:C_0805, F.Cu at (-55.3, 150.8)
- added C13: 100nF, PCM_JLCPCB:C_0805, F.Cu at (-55.3, 153.8)
- added C14: 470uF/25V, Capacitor_SMD:CP_Elec_8x11.9, F.Cu at (-42.3, 148.1)
- added C15: 4.7uF/16V, PCM_JLCPCB:C_CASE-B-3528-21(mm), F.Cu at (-28.4, 130.6)
- added C16: 10uF_16V, PCM_JLCPCB:C_CASE-B-3528-21(mm), F.Cu at (-28.4, 134.9)
- added C17: 0.1uF/25V, PCM_JLCPCB:C_0805, F.Cu at (-55.3, 156.9)
- added C18: 100nF, PCM_JLCPCB:C_0805, F.Cu at (-55.3, 159.9)
- added C19: 4.7uF/16V, Capacitor_Tantalum_SMD:CP_EIA-3216-18_Kemet-A, F.Cu at (-22.4, 159.2)
- added C2: 680uF_35V, Capacitor_SMD:CP_Elec_10x12.5, F.Cu at (26.6, 114.3)
- added C20: 22pF, PCM_JLCPCB:C_0805, F.Cu at (-50.8, 144.7)
- added C21: 22pF, PCM_JLCPCB:C_0805, F.Cu at (-50.8, 147.7)
- added C22: 100nF, PCM_JLCPCB:C_0805, F.Cu at (-50.8, 150.8)
- added C23: 100nF, PCM_JLCPCB:C_0805, F.Cu at (-50.8, 153.8)
- added C24: 100nF, PCM_JLCPCB:C_0805, F.Cu at (-50.8, 156.9)
- added C3: 470nF, PCM_JLCPCB:C_0805, F.Cu at (-55.3, 144.7)
- added C4: 100nF, PCM_JLCPCB:C_0805, F.Cu at (-55.3, 147.7)
- added C5: 220uF_16V, Capacitor_SMD:CP_Elec_6.3x7.7, F.Cu at (34.3, 139.4)
- added C6: 220uF_16V, Capacitor_SMD:CP_Elec_6.3x7.7, F.Cu at (34.3, 147.5)
- added C7: 680uF_35V, Capacitor_SMD:CP_Elec_10x12.5, F.Cu at (26.6, 126.3)
- added C8: 145J400V, Capacitor_THT:C_Rect_L19.0mm_W6.0mm_P15.00mm_MKS4, F.Cu at (-80.7, 147.3)
- added C9: 2200uF/35V, Capacitor_THT:CP_Radial_D18.0mm_P7.50mm, F.Cu at (5.62, 106.0)
- added D1: Blue, LED_THT:LED_D3.0mm, F.Cu at (41.2, 138.0)
- added D10: SM4001, PCM_JLCPCB:D_SMA, F.Cu at (-21.2, 121.2)
- added D11: SM4001, PCM_JLCPCB:D_SMA, F.Cu at (-21.2, 125.8)
- added D12: 1N5824, PCM_JLCPCB:D_SMA, F.Cu at (-21.2, 130.3)
- added D13: 1N5819, PCM_JLCPCB:D_SMA, F.Cu at (-13.1, 98.5)
- added D14: 1N5819, PCM_JLCPCB:D_SMA, F.Cu at (-13.1, 103.0)
- added D15: SM4001, PCM_JLCPCB:D_SMA, F.Cu at (-13.1, 107.6)
- added D16: Red, LED_THT:LED_D3.0mm, F.Cu at (41.2, 149.0)
- added D17: Green, LED_THT:LED_D3.0mm, F.Cu at (41.2, 154.4)
- added D18: SM4001, PCM_JLCPCB:D_SMA, F.Cu at (-13.1, 112.1)
- added D19: SM4001, PCM_JLCPCB:D_SMA, F.Cu at (-13.1, 116.7)
- added D2: 1N5824, PCM_JLCPCB:D_SMA, F.Cu at (-21.2, 98.5)
- added D20: SM4001, PCM_JLCPCB:D_SMA, F.Cu at (-13.1, 121.2)
- added D21: SM4001, PCM_JLCPCB:D_SMA, F.Cu at (-13.1, 125.8)
- added D22: SM4001, PCM_JLCPCB:D_SMA, F.Cu at (-13.1, 130.3)
- added D23: SM4001, PCM_JLCPCB:D_SMA, F.Cu at (-4.97, 98.5)
- added D24: SM4001, PCM_JLCPCB:D_SMA, F.Cu at (-4.97, 103.0)
- added D25: SM4001, PCM_JLCPCB:D_SMA, F.Cu at (-4.97, 107.6)
- added D26: SM4001, PCM_JLCPCB:D_SMA, F.Cu at (-4.97, 112.1)
- added D27: SM4001, PCM_JLCPCB:D_SMA, F.Cu at (-4.97, 116.7)
- added D28: SM4001, PCM_JLCPCB:D_SMA, F.Cu at (-4.97, 121.2)
- added D29: SM4001, PCM_JLCPCB:D_SMA, F.Cu at (-4.97, 125.8)
- added D3: 1N5824, PCM_JLCPCB:D_SMA, F.Cu at (-21.2, 103.0)
- added D4: GREEN, LED_THT:LED_D3.0mm, F.Cu at (41.2, 143.5)
- added D5: SM4001, PCM_JLCPCB:D_SMA, F.Cu at (-21.2, 107.6)
- added D6: SM4001, PCM_JLCPCB:D_SMA, F.Cu at (-21.2, 112.1)
- added D7: SM4001, PCM_JLCPCB:D_SMA, F.Cu at (-21.2, 116.7)
- added D8: GBU8M, Diode_THT:Diode_Bridge_Vishay_GBU, F.Cu at (-21.1, 135.0)
- added D9: GBU8M, Diode_THT:Diode_Bridge_Vishay_GBU, F.Cu at (-21.1, 140.4)
- added DZ1: CMZ12, PCM_JLCPCB:D_SOD-123, F.Cu at (-28.5, 138.8)
- added J1: CT, Connector_PinHeader_2.54mm:PinHeader_1x02_P2.54mm_Vertical, F.Cu at (38.6, 90.4)
- added J10: LOAD 3, TestPoint:TestPoint_Plated_Hole_D5.0mm, F.Cu at (-45.4, 100.2)
- added J11: LOAD 2, TestPoint:TestPoint_Plated_Hole_D5.0mm, F.Cu at (-45.4, 108.3)
- added J12: DISPLAY, Connector_PinHeader_2.54mm:PinHeader_1x12_P2.54mm_Vertical, F.Cu at (43.4, 11.6)
- added J13: TRANS-IN, TerminalBlock_Phoenix:TerminalBlock_Phoenix_PT-1,5-2-5.0-H_1x02_P5.00mm_Horizontal, F.Cu at (37.2, 101.2)
- added J14: TRANS 2-OUT, TerminalBlock_Phoenix:TerminalBlock_Phoenix_PT-1,5-2-5.0-H_1x02_P5.00mm_Horizontal, F.Cu at (37.2, 112.5)
- added J15: TRANS 1-OUT, TerminalBlock_Phoenix:TerminalBlock_Phoenix_PT-1,5-2-5.0-H_1x02_P5.00mm_Horizontal, F.Cu at (37.2, 123.8)
- added J16: N, TestPoint:TestPoint_Plated_Hole_D5.0mm, F.Cu at (-45.4, 116.3)
- added J17: N, TestPoint:TestPoint_Plated_Hole_D5.0mm, F.Cu at (-45.4, 124.4)
- added J18: N, TestPoint:TestPoint_Plated_Hole_D5.0mm, F.Cu at (-37.4, 100.2)
- added J19: N, TestPoint:TestPoint_Plated_Hole_D5.0mm, F.Cu at (-37.4, 108.3)
- added J2: PZEM_LOAD, TerminalBlock:TerminalBlock_MaiXu_MX126-5.0-04P_1x04_P5.00mm, F.Cu at (-21.3, 148.5)
- added J20: N, TestPoint:TestPoint_Plated_Hole_D5.0mm, F.Cu at (-37.4, 116.3)
- added J21: N, TestPoint:TestPoint_Plated_Hole_D5.0mm, F.Cu at (-37.4, 124.4)
- added J22: N, TestPoint:TestPoint_Plated_Hole_D5.0mm, F.Cu at (-29.3, 100.2)
- added J23: N, TestPoint:TestPoint_Plated_Hole_D5.0mm, F.Cu at (-29.3, 108.3)
- added J24: LOAD 1, TestPoint:TestPoint_Plated_Hole_D5.0mm, F.Cu at (-29.3, 116.3)
- added J25: NEPA, TestPoint:TestPoint_Plated_Hole_D5.0mm, F.Cu at (-29.3, 124.4)
- added J3: PZEM_SIG, Connector_PinHeader_2.54mm:PinHeader_1x04_P2.54mm_Vertical, F.Cu at (-33.6, 145.4)
- added J4: USB_C Conn, Connector_PinHeader_2.54mm:PinHeader_1x04_P2.54mm_Vertical, F.Cu at (-29.0, 145.4)
- added J6: INVERTER, TestPoint:TestPoint_Plated_Hole_D5.0mm, F.Cu at (-53.5, 100.2)
- added J7: LOAD 6, TestPoint:TestPoint_Plated_Hole_D5.0mm, F.Cu at (-53.5, 108.3)
- added J8: LOAD 5, TestPoint:TestPoint_Plated_Hole_D5.0mm, F.Cu at (-53.5, 116.3)
- added J9: LOAD 4, TestPoint:TestPoint_Plated_Hole_D5.0mm, F.Cu at (-53.5, 124.4)
- added JP1: ~, Jumper:SolderJumper-3_P1.3mm_Open_Pad1.0x1.5mm, F.Cu at (29.2, 89.9)
- added JP2: ~, Jumper:SolderJumper-3_P1.3mm_Open_Pad1.0x1.5mm, F.Cu at (29.2, 93.7)
- added JP3: ~, Jumper:SolderJumper-2_P1.3mm_Open_Pad1.0x1.5mm, F.Cu at (-17.4, 159.4)
- added K1: 10A RELAY, Relay_THT:Relay_SPDT_Finder_36.11, F.Cu at (14.7, 139.3)
- added K10: 30A RELAY, Relay_THT:Relay_SPDT_RAYEX-L90, F.Cu at (-35.6, 81.2)
- added K11: 30A RELAY, Relay_THT:Relay_SPDT_RAYEX-L90, F.Cu at (-2.25, 23.3)
- added K12: 30A RELAY, Relay_THT:Relay_SPDT_RAYEX-L90, F.Cu at (-2.25, 52.3)
- added K13: 30A RELAY, Relay_THT:Relay_SPDT_RAYEX-L90, F.Cu at (-2.25, 81.2)
- added K2: 30A RELAY, Relay_THT:Relay_SPDT_RAYEX-L90, F.Cu at (-102.3, 23.3)
- added K3: 30A RELAY, Relay_THT:Relay_SPDT_RAYEX-L90, F.Cu at (-102.3, 52.3)
- added K4: 30A RELAY, Relay_THT:Relay_SPDT_RAYEX-L90, F.Cu at (-102.3, 81.2)
- added K5: 30A RELAY, Relay_THT:Relay_SPDT_RAYEX-L90, F.Cu at (-68.9, 23.3)
- added K6: 30A RELAY, Relay_THT:Relay_SPDT_RAYEX-L90, F.Cu at (-68.9, 52.3)
- added K7: 30A RELAY, Relay_THT:Relay_SPDT_RAYEX-L90, F.Cu at (-68.9, 81.2)
- added K8: 30A RELAY, Relay_THT:Relay_SPDT_RAYEX-L90, F.Cu at (-35.6, 23.3)
- added K9: 30A RELAY, Relay_THT:Relay_SPDT_RAYEX-L90, F.Cu at (-35.6, 52.3)
- added L1: 33uH, Inductor_SMD:L_12x12mm_H6mm, F.Cu at (33.8, 16.5)
- added L2: 33uH, Inductor_SMD:L_12x12mm_H6mm, F.Cu at (33.8, 30.7)
- added L3: 33uH, Inductor_SMD:L_12x12mm_H6mm, F.Cu at (33.8, 45.0)
- added OC1: PC817XFP, PCM_JLCPCB:SOP-4_4.4x2.6mm_P1.27mm, F.Cu at (-43.8, 155.1)
- added OC2: PC817XFP, PCM_JLCPCB:SOP-4_4.4x2.6mm_P1.27mm, F.Cu at (-43.8, 159.2)
- added Q1: UMH3N, PCM_JLCPCB:SOT-363_SC-70-6, F.Cu at (34.1, 90.1)
- added Q2: UMH3N, PCM_JLCPCB:SOT-363_SC-70-6, F.Cu at (34.1, 94.0)
- added Q3: ULN2803ADWR, digikey-footprints:SOIC-18_W7.5mm, F.Cu at (5.61, 141.8)
- added Q4: ULN2803ADWR, digikey-footprints:SOIC-18_W7.5mm, F.Cu at (5.61, 154.7)
- added R1: 680k, PCM_JLCPCB:R_0805, F.Cu at (-55.3, 129.9)
- added R10: 10k, PCM_JLCPCB:R_0805, F.Cu at (-50.9, 141.7)
- added R11: 330R, PCM_JLCPCB:R_0805, F.Cu at (-46.5, 129.9)
- added R12: 10k, PCM_JLCPCB:R_0805, F.Cu at (-46.5, 132.8)
- added R13: 1M, Resistor_THT:R_Axial_DIN0207_L6.3mm_D2.5mm_P10.16mm_Horizontal, F.Cu at (-23.7, 155.6)
- added R14: 330R/2W, Resistor_THT:R_Axial_DIN0309_L9.0mm_D3.2mm_P20.32mm_Horizontal, F.Cu at (-81.9, 141.2)
- added R15: 10k, PCM_JLCPCB:R_0805, F.Cu at (-46.5, 135.8)
- added R16: 10k, PCM_JLCPCB:R_0805, F.Cu at (-46.5, 138.7)
- added R17: 10k, PCM_JLCPCB:R_0805, F.Cu at (-46.5, 141.7)
- added R18: 150R, PCM_JLCPCB:R_0805, F.Cu at (-42.0, 129.9)
- added R19: 330R, PCM_JLCPCB:R_0805, F.Cu at (-42.0, 132.8)
- added R2: 680k, PCM_JLCPCB:R_0805, F.Cu at (-55.3, 132.8)
- added R20: 330R, PCM_JLCPCB:R_0805, F.Cu at (-42.0, 135.8)
- added R21: 10k, PCM_JLCPCB:R_0805, F.Cu at (-42.0, 138.7)
- added R22: 10k, PCM_JLCPCB:R_0805, F.Cu at (-42.0, 141.7)
- added R3: 100k, PCM_JLCPCB:R_0805, F.Cu at (-55.3, 135.8)
- added R4: 6.8k, PCM_JLCPCB:R_0805, F.Cu at (-55.3, 138.7)
- added R5: 6.8k, PCM_JLCPCB:R_0805, F.Cu at (-55.3, 141.7)
- added R6: 330R, PCM_JLCPCB:R_0805, F.Cu at (-50.9, 129.9)
- added R7: 680k, PCM_JLCPCB:R_0805, F.Cu at (-50.9, 132.8)
- added R8: 6.8k, PCM_JLCPCB:R_0805, F.Cu at (-50.9, 135.8)
- added R9: 330R, PCM_JLCPCB:R_0805, F.Cu at (-50.9, 138.7)
- added RV1: 10K, Potentiometer_THT:Potentiometer_Bourns_3296W_Vertical, F.Cu at (-88.3, 159.0)
- added SW1: RESET, PCM_JLCPCB:SW_TS-1088-AR02016, F.Cu at (-8.45, 155.8)
- added SW2: FLASH, PCM_JLCPCB:SW_TS-1088-AR02016, F.Cu at (-8.45, 160.3)
- added TP1: TestPoint, TestPoint:TestPoint_Pad_D1.5mm, F.Cu at (-105.3, 140.6)
- added TP10: TestPoint, TestPoint:TestPoint_Pad_D1.5mm, F.Cu at (-101.7, 151.2)
- added TP11: TestPoint, TestPoint:TestPoint_Pad_D1.5mm, F.Cu at (-101.7, 154.8)
- added TP12: TestPoint, TestPoint:TestPoint_Pad_D1.5mm, F.Cu at (-101.7, 158.3)
- added TP13: TestPoint, TestPoint:TestPoint_Pad_D1.5mm, F.Cu at (-98.2, 140.6)
- added TP14: TestPoint, TestPoint:TestPoint_Pad_D1.5mm, F.Cu at (-98.2, 144.1)
- added TP15: TestPoint, TestPoint:TestPoint_Pad_D1.5mm, F.Cu at (-98.2, 147.7)
- added TP16: TestPoint, TestPoint:TestPoint_Pad_D1.5mm, F.Cu at (-98.2, 151.2)
- added TP17: TestPoint, TestPoint:TestPoint_Pad_D1.5mm, F.Cu at (-98.2, 154.8)
- added TP2: TestPoint, TestPoint:TestPoint_Pad_D1.5mm, F.Cu at (-105.3, 144.1)
- added TP3: TestPoint, TestPoint:TestPoint_Pad_D1.5mm, F.Cu at (-105.3, 147.7)
- added TP4: TestPoint, TestPoint:TestPoint_Pad_D1.5mm, F.Cu at (-105.3, 151.2)
- added TP5: TestPoint, TestPoint:TestPoint_Pad_D1.5mm, F.Cu at (-105.3, 154.8)
- added TP6: TestPoint, TestPoint:TestPoint_Pad_D1.5mm, F.Cu at (-105.3, 158.3)
- added TP7: TestPoint, TestPoint:TestPoint_Pad_D1.5mm, F.Cu at (-101.7, 140.6)
- added TP8: TestPoint, TestPoint:TestPoint_Pad_D1.5mm, F.Cu at (-101.7, 144.1)
- added TP9: TestPoint, TestPoint:TestPoint_Pad_D1.5mm, F.Cu at (-101.7, 147.7)
- added U1: LM2596S-3.3V, PCM_JLCPCB:TO-263-5_L10.2-W8.9-P1.70-TL, F.Cu at (33.5, 58.1)
- added U2: LM2596S-12, PCM_JLCPCB:TO-263-5_L10.2-W8.9-P1.70-TL, F.Cu at (33.5, 70.1)
- added U3: ESP32-WROOM, RF_Module:ESP32-WROOM-32E, F.Cu at (-82.3, 124.7)
- added U4: LM2596S-5V, PCM_JLCPCB:TO-263-5_L10.2-W8.9-P1.70-TL, F.Cu at (33.5, 82.1)
- added U5: AMS1117-3.3, PCM_JLCPCB:SOT-223-3_L6.5-W3.4-P2.30-LS7.0-BR, F.Cu at (-63.4, 155.1)
- added U6: PCA9555D, Package_SO:SOIC-24W_7.5x15.4mm_P1.27mm, F.Cu at (-89.9, 147.4)
- added U7: CH340C, PCM_JLCPCB:SOIC-16_3.9x9.9mm_P1.27mm, F.Cu at (-35.6, 134.3)
- added Y1: 12MHz, PCM_JLCPCB:CRYSTAL-SMD_L11.5-W4.8-LS12.7, F.Cu at (-75.8, 154.1)
- moved J13 204.4 mm to (0.25, 186.6)
- moved J6 204.4 mm to (-61.3, 175.2)
Other:
- board outline added: 138.4 x 97.3 mm

Commit message: update from home
Parts:
- removed the J13 at (0.25, 186.6)
- removed the J6 at (-61.3, 175.2)
- moved K2 378.9 mm to (273.2, 74.2), turned to -90 degrees
- moved K3 346.0 mm to (243.0, 74.2), turned to -90 degrees
- moved K8 320.3 mm to (273.1, 108.8), turned to -90 degrees
- moved J7 318.8 mm to (263.5, 142.5)
- moved J20 316.8 mm to (278.4, 142.5)
- moved K4 315.3 mm to (212.9, 74.2), turned to -90 degrees
- moved J8 288.4 mm to (233.8, 142.5)
- moved J21 286.6 mm to (248.6, 142.5)
- moved K9 284.2 mm to (243.0, 108.8), turned to -90 degrees
- moved J19 258.5 mm to (218.9, 142.5)
- moved J9 258.1 mm to (204.0, 142.5)
- moved K5 256.8 mm to (182.8, 74.1), turned to -90 degrees
- moved K10 250.0 mm to (212.9, 108.8), turned to -90 degrees
- moved J18 230.4 mm to (189.2, 142.5)
- moved J3 226.9 mm to (174.9, 55.9), turned to 180 degrees
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Other:
- board size 138.4 x 97.3 mm -> 200 x 136.9 mm
- copper layers 2 -> 4

Commit message: update from work
Parts:
- removed D15: SM4001, PCM_JLCPCB:D_SMA
- added C25: 100nF, PCM_JLCPCB:C_0805, F.Cu at (226.4, 41.2)
- added REF**: M3, MountingHole:MountingHole_3.2mm_M3_Pad, F.Cu at (245.0, 28.0)
- added REF**: M3, MountingHole:MountingHole_3.2mm_M3_Pad, F.Cu at (54.5, 28.1)
- added REF**: M3, MountingHole:MountingHole_3.2mm_M3_Pad, F.Cu at (245.3, 151.1)
- added REF**: M3, MountingHole:MountingHole_3.2mm_M3_Pad, F.Cu at (54.5, 150.8)
- C17, C23, C24, D18, D19, D20, D21, D22, D23, D24, D25, D26, D27, D28, D29, Q3, Q4, R15, R16, R17, U6: moved to B.Cu
- moved TP10 374.4 mm to (240.8, 11.7)
- moved TP4 374.4 mm to (240.8, 4.58)
- moved TP9 374.4 mm to (240.8, 8.13)
- moved TP5 366.9 mm to (237.2, 10.6)
- moved TP6 365.7 mm to (233.6, 8.83)
- moved TP8 362.8 mm to (236.5, 14.5)
- moved TP11 359.4 mm to (223.0, 4.33)
- moved TP12 359.4 mm to (219.5, 4.33)
- moved TP7 357.8 mm to (232.5, 14.5)
- moved TP16 357.7 mm to (229.8, 9.80)
- moved TP17 357.7 mm to (229.8, 13.4)
- moved TP1 356.8 mm to (232.1, 5.43)
- moved TP13 356.8 mm to (228.6, 5.43)
- moved TP14 350.4 mm to (225.2, 9.15)
- moved TP15 350.4 mm to (225.2, 12.7)
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- renumbered J25 to J1, J17 to J10, J3 to J11, J18 to J12, J19 to J13, J4 to J14, J13 to J17, J14 to J18, J12 to J19, J6 to J2, J7 to J20, J8 to J21, J9 to J22, J10 to J23, J11 to J24, J24 to J25, J1 to J3, J20 to J4, J21 to J5, J2 to J6, J22 to J7, J23 to J8, J16 to J9, TP13 to TP1, TP5 to TP10, TP12 to TP11, TP6 to TP12, TP7 to TP13, TP8 to TP16, TP9 to TP17, TP1 to TP2, TP2 to TP3, TP3 to TP4, TP10 to TP5, TP11 to TP6, TP16 to TP7, TP17 to TP8, TP4 to TP9
Other:
- board size 200 x 136.9 mm -> 198.1 x 130.3 mm

Commit message: update from home
Routing:
- net +12V: track 0.00 -> 25.4 mm, vias 0 -> 34
- net Net-(D11-A): track 0.00 -> 4.48 mm
- net Net-(D10-A): track 0.00 -> 4.45 mm
- net +3.3V: track 0.00 -> 1.47 mm, vias 0 -> 36
- net GND: vias 0 -> 1
- net +5V: vias 0 -> 15
- added copper zone on B.Cu, net +12V
- added copper zone on In2.Cu, net +12V
- added copper zone on B.Cu, net GND
- added copper zone on F.Cu, net GND
Other:
- outline, holes or cut-outs redrawn

Commit message: update from work
Parts:
- removed J12, J13, J4, J5, J7, J8: N, TestPoint:TestPoint_Plated_Hole_D5.0mm
- moved R2 11.5 mm to (224.5, 74.0)
- moved J20 10.2 mm to (232.8, 148.0)
- moved J21 10.1 mm to (203.0, 148.0)
- moved J22 9.95 mm to (173.1, 148.0)
- moved J23 9.86 mm to (143.3, 148.0)
- moved R7 9.81 mm to (218.7, 86.7)
- moved R1 9.81 mm to (216.0, 86.7)
- moved J24 9.76 mm to (113.4, 148.0)
- moved J25 9.66 mm to (83.6, 148.0)
- moved R8 9.21 mm to (158.4, 85.7), turned to -90 degrees
- moved R4 8.99 mm to (155.6, 85.7), turned to -90 degrees
- moved R5 8.63 mm to (161.2, 85.7), turned to -90 degrees
- moved Q1 7.21 mm to (186.4, 82.9)
- moved R9 7.21 mm to (186.5, 86.8)
- moved D19 3.67 mm to (190.6, 82.6)
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Connections:
- net Net-(J20-Pin_1) renamed /LOAD6
- net Net-(J21-Pin_1) renamed /LOAD5
- net Net-(J22-Pin_1) renamed /LOAD4
- net Net-(J23-Pin_1) renamed /LOAD3
- net Net-(J24-Pin_1) renamed /LOAD2
- net Net-(J25-Pin_1) renamed /LOAD1
- net Net-(K10-Pad11A) renamed /SELECT4
- net Net-(K11-Pad11A) renamed /SELECT3
- net Net-(K12-Pad11A) renamed /SELECT2
- net Net-(K13-Pad11A) renamed /SELECT1
- net Net-(K2-Pad11A) renamed /SELECT6
- net Net-(K3-Pad11A) renamed /SELECT5
Routing:
- net /RD1C5: track 0.00 -> 179.1 mm, vias 0 -> 4
- net /RD2C1: track 0.00 -> 130.2 mm, vias 0 -> 2
- net /RD1C6: track 0.00 -> 122.8 mm, vias 0 -> 2
- net /RD1C7: track 0.00 -> 119.7 mm, vias 0 -> 2
- net /RD2C3: track 0.00 -> 76.1 mm, vias 0 -> 2
- net /RD1C8: track 0.00 -> 74.2 mm, vias 0 -> 4
- net /RD2C2: track 0.00 -> 46.6 mm, vias 0 -> 2
- net /RD2C4: track 0.00 -> 32.0 mm, vias 0 -> 2
- net /CT +: track 0.00 -> 12.7 mm
- net /RD1C3: track 0.00 -> 10.8 mm, vias 0 -> 2
- net /CT -: track 0.00 -> 10.6 mm
- net /RD1C4: track 0.00 -> 9.67 mm, vias 0 -> 2
- net +12V: track 25.4 -> 33.2 mm
- net /RD1C2: track 0.00 -> 6.91 mm, vias 0 -> 2
- net /RD1C1: vias 0 -> 2
- added copper zone on F.Cu, net +3.3V
- added copper zone on In1.Cu, net +3.3V
- added copper zone on B.Cu, net /LOAD1
- added copper zone on F.Cu, net /LOAD1
- added copper zone on B.Cu, net /LOAD2
- added copper zone on F.Cu, net /LOAD2
- added copper zone on B.Cu, net /LOAD3
- added copper zone on F.Cu, net /LOAD3
- added copper zone on B.Cu, net /LOAD4
- added copper zone on F.Cu, net /LOAD4
- added copper zone on B.Cu, net /LOAD5
- added copper zone on F.Cu, net /LOAD5
- added copper zone on B.Cu, net /LOAD6
- added copper zone on F.Cu, net /LOAD6
- added copper zone on B.Cu, net /SELECT1
- added copper zone on F.Cu, net /SELECT1
- added copper zone on B.Cu, net /SELECT2
- added copper zone on F.Cu, net /SELECT2
- added copper zone on B.Cu, net /SELECT3
- added copper zone on F.Cu, net /SELECT3
- added copper zone on B.Cu, net /SELECT4
- added copper zone on F.Cu, net /SELECT4
- added copper zone on B.Cu, net /SELECT5
- added copper zone on F.Cu, net /SELECT5
- added copper zone on B.Cu, net /SELECT6
- added copper zone on F.Cu, net /SELECT6

Commit message: update from work
Parts:
- removed J9: N, TestPoint:TestPoint_Plated_Hole_D5.0mm
- D18, D19, D20, D21, D22, D23, D24, D25, D26, D27, D28, D29: moved to F.Cu
- moved D29 29.7 mm to (67.8, 113.5)
- moved D25 29.2 mm to (188.3, 113.5)
- moved D28 29.0 mm to (98.0, 113.5)
- moved D27 28.8 mm to (128.2, 113.5)
- moved D26 28.6 mm to (158.4, 113.5)
- moved D24 27.6 mm to (218.9, 113.5)
- moved J10 19.2 mm to (58.9, 74.5)
- moved J1 11.7 mm to (58.7, 90.8)
- moved Q1 4.91 mm to (188.3, 87.4)
- moved R9 4.73 mm to (188.3, 91.2)
- moved J2 4.67 mm to (58.7, 118.1)
- moved D21 2.93 mm to (128.1, 79.1)
- moved D19 2.44 mm to (188.2, 82.0)
- moved J3 2.43 mm to (57.2, 59.4)
- moved D23 2.21 mm to (67.8, 79.2)
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Connections:
- net Net-(J11-Pin_2) renamed /TXP
- net Net-(J11-Pin_3) renamed /RXN
Routing:
- net +12V: track 33.2 -> 571.4 mm, vias 34 -> 42
- net /NEPA: track 0.00 -> 81.9 mm
- net /N: track 0.00 -> 24.8 mm
- net /RD2C3: track 76.1 -> 95.4 mm
- net /RD2C2: track 46.6 -> 64.3 mm, vias 2 -> 4
- net /RD1C7: track 119.7 -> 132.9 mm, vias 2 -> 3
- net /RD1C8: track 74.2 -> 86.7 mm, vias 4 -> 2
- net /RD1C3: track 10.8 -> 0.00 mm, vias 2 -> 1
- net /RD2C1: track 130.2 -> 120.3 mm, vias 2 -> 4
- net /RD1C4: track 9.67 -> 0.00 mm, vias 2 -> 1
- net /RD1C6: track 122.8 -> 115.8 mm
- net /RD1C2: track 6.91 -> 0.00 mm, vias 2 -> 1
- net /RD2C4: track 32.0 -> 36.7 mm
- net /RD1C5: track 179.1 -> 175.1 mm
- net Net-(Q1A-E1): track 0.00 -> 2.61 mm
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- added copper zone on F.Cu, net +12V
- added copper zone on In1.Cu, net +12V
- added copper zone on B.Cu, net /INVERTER
- added copper zone on B.Cu, net /NEPA
- removed copper zone on B.Cu, net /SELECT1
- removed copper zone on B.Cu, net /SELECT2
- removed copper zone on B.Cu, net /SELECT3
- removed copper zone on B.Cu, net /SELECT4
- removed copper zone on B.Cu, net /SELECT5
- removed copper zone on B.Cu, net /SELECT6
Other:
- outline, holes or cut-outs redrawn

Commit message: update from home
Routing:
- net /RD1C1: track 0.00 -> 261.6 mm, vias 1 -> 2
- net +12V: track 571.4 -> 825.5 mm, vias 42 -> 39
- net /RD1C3: track 0.00 -> 218.3 mm, vias 1 -> 2
- net /RD1C2: track 0.00 -> 178.1 mm, vias 1 -> 2
- net /RD1C4: track 0.00 -> 141.7 mm, vias 1 -> 2
- net /NEPA: track 81.9 -> 99.5 mm
- net /RD2C3: track 95.4 -> 97.8 mm
- net /RD2C4: track 36.7 -> 39.0 mm
- net /RD2C2: track 64.3 -> 66.6 mm
- net /RD1C6: track 115.8 -> 114.3 mm
- net /RD1C5: track 175.1 -> 173.8 mm, vias 4 -> 6
- net /RD1C8: track 86.7 -> 87.4 mm
- net /RD1C7: vias 3 -> 2
Other:
- outline, holes or cut-outs redrawn

Commit message: update from work
Parts:
- added C26: 10uF_16V, PCM_JLCPCB:C_CASE-B-3528-21(mm), F.Cu at (129.6, 86.2)
- added C27: 10uF_16V, PCM_JLCPCB:C_CASE-B-3528-21(mm), F.Cu at (125.9, 86.2)
- added D15: SM4007PL, PCM_JLCPCB:D_SMA, B.Cu at (221.4, 66.9)
- added D30: SM4007PL, PCM_JLCPCB:D_SMA, B.Cu at (221.5, 62.5)
- moved R2 34.5 mm to (191.5, 84.0), turned to 90 degrees
- moved D18 1.39 mm to (220.2, 79.1)
- moved C13 1.30 mm to (161.2, 43.2)
Connections:
- R1 pad 2: /NEPA -> Net-(D15-K)
- R2 pad 2: /INVERTER -> Net-(D30-K)
Routing:
- net VCC3: track 0.00 -> 183.5 mm, vias 0 -> 1
- net Net-(Q3-IN8): track 0.00 -> 117.2 mm, vias 0 -> 2
- net Net-(Q3-IN7): track 0.00 -> 114.6 mm, vias 0 -> 2
- net Net-(Q3-IN6): track 0.00 -> 111.8 mm, vias 0 -> 2
- net Net-(Q4-IN1): track 0.00 -> 108.3 mm, vias 0 -> 2
- net Net-(Q4-IN2): track 0.00 -> 106.5 mm, vias 0 -> 2
- net Net-(Q4-IN3): track 0.00 -> 104.8 mm, vias 0 -> 2
- net Net-(Q4-IN4): track 0.00 -> 103.1 mm, vias 0 -> 2
- net /N: track 24.8 -> 97.7 mm, vias 0 -> 3
- net +5V: track 0.00 -> 65.2 mm, vias 15 -> 18
- net /INVERTER_SENSE: track 0.00 -> 36.7 mm, vias 0 -> 2
- net /NEPA_SENSE: track 0.00 -> 35.3 mm, vias 0 -> 2
- net Net-(Q1A-C1): track 0.00 -> 32.7 mm, vias 0 -> 3
- net /NEPA: track 99.5 -> 123.2 mm
- net +12V: track 825.5 -> 848.0 mm
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- added copper zone on In2.Cu, net +3.3V
- added copper zone on F.Cu, net +5V
- added copper zone on In2.Cu, net +5V
- removed copper zone on In1.Cu, net +12V
Other:
- outline, holes or cut-outs redrawn
