File: ESP32/Smart Home Energy Management System/Smart Home Energy Management System.kicad_pcb (KiCad board)
At the start: 4 copper layers, 198.1 x 130.3 mm, 154 parts, among them J1 NEPA, J10 N, J11 PZEM_SIG, J14 USB_C Conn, J15 TRANS 1-OUT, J17 TRANS-IN, J18 TRANS 2-OUT, J19 DISPLAY, J2 INVERTER, J20 LOAD 6, J21 LOAD 5, J22 LOAD 4, J23 LOAD 3, J24 LOAD 2, J25 LOAD 1, J3 CT, J6 PZEM_LOAD, K1 10A RELAY, K10 30A RELAY, K11 30A RELAY, K12 30A RELAY, K13 30A RELAY, K2 30A RELAY, K3 30A RELAY, K4 30A RELAY, K5 30A RELAY, K6 30A RELAY, K7 30A RELAY, K8 30A RELAY, K9 30A RELAY, Q1 UMH3N, Q2 UMH3N, Q3 ULN2803ADWR, Q4 ULN2803ADWR, SW1 RESET, SW2 FLASH, U1 LM2596S-3.3V, U2 LM2596S-12, U3 ESP32-WROOM, U4 LM2596S-5V, U5 AMS1117-3.3, U6 PCA9555D, U7 CH340C, Y1 12MHz

Commit message: update from work
Parts:
- moved TP4 148.7 mm to (96.3, 40.0)
- moved D12 52.5 mm to (137.4, 67.0), turned to -90 degrees
- moved TP9 33.2 mm to (207.7, 11.0)
- moved TP5 33.0 mm to (204.2, 11.0)
- moved TP10 31.6 mm to (211.2, 0.35)
- moved TP8 29.6 mm to (207.7, 7.45)
- moved TP1 28.4 mm to (204.2, 0.35)
- moved TP6 27.3 mm to (207.7, 0.35)
- moved TP7 27.0 mm to (207.7, 3.90)
- moved TP13 18.2 mm to (211.2, 11.0)
- moved TP16 15.2 mm to (214.8, 7.45)
- moved TP17 15.2 mm to (214.8, 11.0)
- moved TP2 14.8 mm to (204.2, 3.90)
- moved TP3 14.8 mm to (204.2, 7.45)
- moved TP14 13.7 mm to (214.8, 0.35)
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Routing:
- net Net-(Q3-IN5): track 0.00 -> 111.9 mm, vias 0 -> 2
- net Net-(Q3-IN4): track 0.00 -> 109.3 mm, vias 0 -> 2
- net Net-(Q3-IN3): track 0.00 -> 108.3 mm, vias 0 -> 2
- net Net-(Q3-IN1): track 0.00 -> 108.0 mm, vias 0 -> 2
- net Net-(Q3-IN2): track 0.00 -> 105.2 mm, vias 0 -> 2
- net +5V: track 65.2 -> 162.6 mm, vias 18 -> 15
- net Net-(D3-K): track 0.00 -> 91.9 mm, vias 0 -> 6
- net VCC1: track 0.00 -> 90.5 mm, vias 0 -> 5
- net Net-(U2-~{ON}/OFF): track 0.00 -> 72.6 mm, vias 0 -> 4
- net VCC2: track 12.8 -> 63.4 mm, vias 1 -> 6
- net /GPIO2: track 0.00 -> 35.9 mm, vias 0 -> 2
- net Net-(D11-A): track 4.48 -> 32.3 mm, vias 0 -> 1
- net /N: track 97.7 -> 123.7 mm
- net Net-(D12-K): track 0.00 -> 25.9 mm, vias 0 -> 2
- net /CONST: track 0.00 -> 24.7 mm
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- added copper zone on B.Cu, net +3.3V
- added copper zone on B.Cu, net VCC1
- added copper zone on F.Cu, net VCC1
- added copper zone on In2.Cu, net VCC1
- added copper zone on In2.Cu, net VCC2
Other:
- outline, holes or cut-outs redrawn

Commit message: update from home
Parts:
- removed TP1, TP10, TP11, TP12, TP13, TP15, TP16, TP17, TP2, TP3, TP5, TP6, TP9: TestPoint, TestPoint:TestPoint_Pad_D1.5mm
- moved TP8 63.7 mm to (242.4, 60.8), turned to 90 degrees
- moved TP7 63.2 mm to (235.0, 60.9), turned to 90 degrees
- moved TP14 58.0 mm to (194.1, 54.5), turned to 90 degrees
- moved J14 1.31 mm to (226.9, 27.6)
- moved C18 0.67 mm to (214.9, 28.0)
- moved C14 0.18 mm to (237.6, 66.7)
Connections:
- net /RXN renamed Net-(J11-Pin_3)
- net /TXP renamed Net-(J11-Pin_2)
- net Net-(J14-Pin_2) renamed /D+
- net Net-(J14-Pin_3) renamed /D-
Routing:
- net /GPIO1/TX: track 5.40 -> 191.1 mm, vias 0 -> 4
- net /GPIO3/RX: track 12.7 -> 181.6 mm, vias 0 -> 4
- net /GPIO17: track 0.00 -> 89.4 mm, vias 0 -> 1
- net /IND_LED: track 0.00 -> 87.5 mm, vias 0 -> 3
- net /N: track 123.7 -> 207.9 mm
- net /GPIO22/SCL: track 8.41 -> 91.7 mm, vias 0 -> 5
- net /GPIO16: track 0.00 -> 77.0 mm, vias 0 -> 1
- net /NEPA_SENSE: track 35.0 -> 110.7 mm, vias 2 -> 6
- net /GPIO21/SDA: track 8.35 -> 81.5 mm, vias 0 -> 3
- net /INVERTER: track 3.93 -> 68.0 mm, vias 0 -> 2
- net /INVERTER_SENSE: track 36.7 -> 93.2 mm, vias 2 -> 4
- net Net-(D5-A): track 0.00 -> 53.7 mm, vias 0 -> 2
- net /GPIO0: track 3.33 -> 51.9 mm, vias 0 -> 3
- net +3.3V: track 17.8 -> 63.6 mm, vias 35 -> 32
- net Net-(D30-K): track 0.00 -> 45.5 mm, vias 0 -> 3
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Other:
- outline, holes or cut-outs redrawn

Commit message: update from home
Parts:
- R13: footprint Resistor_THT:R_Axial_DIN0207_L6.3mm_D2.5mm_P10.16mm_Horizontal -> Resistor_THT:R_Axial_DIN0207_L6.3mm_D2.5mm_P7.62mm_Horizontal
- moved R13 0.98 mm to (56.4, 39.9)
- moved C13 0.43 mm to (161.2, 42.8)
Routing:
- net /N: track 207.9 -> 351.6 mm, vias 3 -> 2
- net /GPIO23/MOSI: track 1.78 -> 92.1 mm
- net Net-(U6-IO1_5): track 0.00 -> 82.9 mm, vias 0 -> 1
- net /GPIO18/SCK: track 0.00 -> 77.8 mm, vias 0 -> 1
- net /GPIO5/CS: track 0.00 -> 72.7 mm, vias 0 -> 1
- net /GPIO26: track 18.2 -> 72.1 mm
- net Net-(D12-K): track 25.9 -> 70.5 mm, vias 2 -> 4
- net Net-(D2-K): track 25.8 -> 70.0 mm, vias 2 -> 4
- net /GPIO25: track 23.1 -> 66.8 mm, vias 2 -> 4
- net /GPIO17: track 89.4 -> 125.8 mm, vias 1 -> 3
- net /GPIO16: track 77.0 -> 111.4 mm, vias 1 -> 3
- net /TRANS-IN: track 0.00 -> 31.8 mm, vias 0 -> 2
- net Net-(D14-A): track 10.6 -> 41.4 mm, vias 0 -> 3
- net Net-(OC2-Pad1): track 0.00 -> 22.7 mm, vias 0 -> 2
- net +3.3V: track 63.6 -> 82.4 mm
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Other:
- board size 198.1 x 130.3 mm -> 198.1 x 130.8 mm

Commit message: update from work
Parts:
- U3: value ESP32-WROOM -> ESP32
- moved REF** 1.47 mm to (244.2, 150.1)
- moved REF** 0.82 mm to (55.2, 150.4)
- moved REF** 0.74 mm to (55.2, 28.1)
- moved REF** 0.55 mm to (244.5, 28.2)
- renumbered J17 to XFORMER_IN, J18 to XFORMER_OUT1, J15 to XFORMER_OUT2
Routing:
- net /N: track 351.6 -> 353.2 mm
- net Net-(D30-K): track 44.5 -> 45.1 mm
Other:
- outline, holes or cut-outs redrawn
- board text added: "+"
- board text added: "+3V3"
- board text added: "+5V"
- board text added: "-"
- board text added: "A"
- board text added: "B"
- board text added: "CT"
- board text added: "D+"
- board text added: "D-"
- board text added: "G"
- board text added: "INVERTER"
- board text added: "LOAD 1"
- board text added: "LOAD 2"
- board text added: "LOAD 3"
- board text added: "LOAD 4"
- board text added: "LOAD 5"
- board text added: "LOAD 6"
- board text added: "M3"
- board text added: "N"
- board text added: "NEPA"
- board text added: "P3"
- board text added: "P4"
- board text added: "P5"
- board text added: "P6"
- board text added: "PZEM-004T"
- board text added: "RX"
- board text added: "SW"
- board text added: "TX"
