File: ESP32/Solar_Powered Egg_Incubator/hardware/Solar_Powered_Egg_Incubator.kicad_sch (KiCad schematic)
At the start: 102 parts, among them J1 FAN, J2 SPINNER, J23 USB_C Conn, J3 BMS, J4 RTC, J42 Ultra Sonic, J47 SCREEN, J5 AHT20, J6 HUMIDIFIER, J7 HEATER, J8 LEVELS, K4 RELAY, K5 RELAY, K6 RELAY, Q2 UMH3N, Q9 TIP41, SW4 RESET, SW5 FLASH, SW6 RotaryEncoder, U1 LM2596S-3.3V, U3 LM2596S-5V, U5 AMS1117-3.3, U7 ESP32-WROOM, U8 CH340C, Y2 12MHz

Commit message: update from home
Parts:
- JP2, JP3, JP4, JP5: value ~ -> (none)
